File: PCB/ESP32_MotorDriver/ESP32_MotorDriver.kicad_pcb (KiCad board)
At the start: 4 copper layers, 30.5 x 58.4 mm, 39 parts, among them J1 USB_C_Receptacle_USB2.0, J2 Conn_01x06, J4 Conn_01x05, J6 Conn_01x07, J7 Conn_01x17, Q1 SSM3J338R_LF, SW1 EN, SW2 BOOT, U1 ESP32-S2-SOLO-N4, U2 D3V3XA4B10LP, U4 TB6612FNG, U5 AP63203WU

Commit message: actual _v01
Issue with files being copied - these should be good
Parts:
- removed R10, R9: 4k7, Resistor_SMD:R_0402_1005Metric_Pad0.72x0.64mm_HandSolder
- added D3: SMAJ12A, Diode_SMD:D_SMA, F.Cu at (133.5, 80.0)
- added F2: Polyfuse 500mA, Fuse:Fuse_0805_2012Metric_Pad1.15x1.40mm_HandSolder, B.Cu at (124.5, 66.0)
- added R5: 22R, Resistor_SMD:R_0402_1005Metric_Pad0.72x0.64mm_HandSolder, F.Cu at (124.5, 66.0)
- added R6: 22R, Resistor_SMD:R_0402_1005Metric_Pad0.72x0.64mm_HandSolder, F.Cu at (124.5, 65.0)
- D1, D2: value D_Schottky -> SS14HE
- F1: value Polyfuse 4A -> Polyfuse 3A; footprint Fuse:Fuse_0805_2012Metric_Pad1.15x1.40mm_HandSolder -> Fuse:Fuse_1812_4532Metric_Pad1.30x3.40mm_HandSolder
- Q1: value SSM3J338R_LF -> AO3407A; footprint SSM3J338R_LF:SOT-23F_TOS -> Package_TO_SOT_SMD:SOT-23
- SW1: value EN -> RESET
- U2: value D3V3XA4B10LP -> USBLC6-2SC6; footprint Package_DFN_QFN:Diodes_UDFN-10_1x2.5mm_P0.5mm -> Package_TO_SOT_SMD:SOT-23-6
- moved C15 5.21 mm to (136.4, 80.0), turned to 90 degrees
- moved C12 3.51 mm to (121.2, 78.6)
- moved C7 3.01 mm to (126.0, 79.2), turned to 0 degrees
- moved C11 2.98 mm to (120.4, 80.3)
- moved F1 1.53 mm to (119.1, 83.3)
- moved R11 1.48 mm to (119.0, 88.1), turned to 0 degrees
- moved C14 1.27 mm to (126.6, 74.8), turned to 0 degrees
- moved U2 0.99 mm to (124.6, 70.4)
- moved C4 0.64 mm to (120.0, 79.5)
- moved Q1 0.25 mm to (118.5, 87.9), turned to -90 degrees
Connections:
- net /MISO renamed /IO12
- net /MOSI renamed /IO13
- net /SCK renamed /IO11
- net /SCL renamed /IO33
- net /SDA renamed /IO34
- F1 pad 1: Net-(F1-Pad1) -> Net-(Q1-S)
- J1 pad A4: VBUS -> Net-(F2-Pad1)
- J1 pad A9: VBUS -> Net-(F2-Pad1)
- J1 pad B4: VBUS -> Net-(F2-Pad1)
- J1 pad B9: VBUS -> Net-(F2-Pad1)
- Q1 pad 2: Vbatt -> Net-(Q1-S)
- Q1 pad 3: Net-(F1-Pad1) -> Vbatt
- U1 pad 13: /USB_N -> /USB_N_ESP
- U1 pad 14: /USB_P -> /USB_P_ESP
- U2 pad 1: VBUS -> /USB_N
- U2 pad 2: /USB_N -> GND
- U2 pad 3: GND -> /USB_P
- U2 pad 6: VBUS -> /USB_N
Routing:
- net Net-(F2-Pad1): track 0.00 -> 16.7 mm, vias 0 -> 4
- net /USB_N_ESP: track 0.00 -> 12.3 mm
- net VBUS: track 30.0 -> 19.1 mm, vias 4 -> 1
- net /USB_P_ESP: track 0.00 -> 9.90 mm
- net /USB_N: track 24.3 -> 14.8 mm
- net /USB_P: track 24.0 -> 16.6 mm
- net +3V3: track 118.0 -> 111.3 mm
- net Net-(Q1-S): track 0.00 -> 3.03 mm
- net Net-(F1-Pad1): track 2.49 -> 0.00 mm
- net /IO34: track 19.6 -> 17.7 mm
- net /IO33: track 22.7 -> 20.8 mm
- net GND: track 27.3 -> 29.1 mm
- net Net-(Q1-G): track 1.63 -> 3.24 mm
- net /IO3: track 30.7 -> 31.8 mm
- net /IO9: track 32.6 -> 33.7 mm
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Other:
- outline, holes or cut-outs redrawn
- board text added: "13.5V"
- board text added: "MAX"

Commit message: BOB v02
Submitted for manufacturer with a few minor fixes from v01. 3V3 to LineFollower array, New footprint for Motor connections and a switch added for power on/off
Parts:
- D1, D2: footprint Diode_SMD:D_SOD-323F -> _diodes:D_SOD-323HE_SS14HE
